File: tht-heatsink/kicad/to263-prototype.kicad_pcb (KiCad board)
At the start: 2 copper layers, 91.4 x 66 mm, 15 parts, among them J1 Conn_01x01, J2 Conn_01x01, J3 Conn_01x01, J4 Conn_01x01, J5 Conn_01x01, J6 Conn_01x01, J7 Conn_01x01, J8 Conn_01x01, U1 Conn_01x07

Commit message: tht heatsink gerbers
Other:
- board text added: "GND"
- board text added: "https://github.com/ uw-madison-chem-shops/ to263-prototype"
Changed lines of the file:
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@@
       (outputformat 1)
       (mirror false)
-      (drillshape 1)
+      (drillshape 0)
       (scaleselection 1)
-      (outputdirectory "")
+      (outputdirectory "../gerber")
     )
   )
@@
     (pad "4" smd roundrect (at -7.65 0 90) (size 4.6 0.8) (layers "F.Cu" "F.Paste" "F.Mask") (roundrect_rratio 0.25)
       (net 4 "Net-(J4-Pin_1)") (pinfunction "Pin_4") (pintype "passive"))
-    (pad "4" smd roundrect (at -0.925 -2.775 90) (size 4.55 5.25) (layers "F.Cu" "F.Paste") (roundrect_rratio 0.054945)
+    (pad "4" smd roundrect (at -0.925 -2.775 90) (size 4.55 5.25) (layers "F.Cu" "F.Paste") (roundrect_rratio 0.05494505495)
       (net 4 "Net-(J4-Pin_1)") (pinfunction "Pin_4") (pintype "passive"))
-    (pad "4" smd roundrect (at -0.925 2.775 90) (size 4.55 5.25) (layers "F.Cu" "F.Paste") (roundrect_rratio 0.054945)
+    (pad "4" smd roundrect (at -0.925 2.775 90) (size 4.55 5.25) (layers "F.Cu" "F.Paste") (roundrect_rratio 0.05494505495)
       (net 4 "Net-(J4-Pin_1)") (pinfunction "Pin_4") (pintype "passive"))
-    (pad "4" smd roundrect (at 1.5 0 90) (size 9.4 10.8) (layers "F.Cu" "F.Mask") (roundrect_rratio 0.026596)
+    (pad "4" smd roundrect (at 1.5 0 90) (size 9.4 10.8) (layers "F.Cu" "F.Mask") (roundrect_rratio 0.02659595745)
       (net 4 "Net-(J4-Pin_1)") (pinfunction "Pin_4") (pintype "passive"))
-    (pad "4" smd roundrect (at 3.925 -2.775 90) (size 4.55 5.25) (layers "F.Cu" "F.Paste") (roundrect_rratio 0.054945)
+    (pad "4" smd roundrect (at 3.925 -2.775 90) (size 4.55 5.25) (layers "F.Cu" "F.Paste") (roundrect_rratio 0.05494505495)
       (net 4 "Net-(J4-Pin_1)") (pinfunction "Pin_4") (pintype "passive"))
-    (pad "4" smd roundrect (at 3.925 2.775 90) (size 4.55 5.25) (layers "F.Cu" "F.Paste") (roundrect_rratio 0.054945)
+    (pad "4" smd roundrect (at 3.925 2.775 90) (size 4.55 5.25) (layers "F.Cu" "F.Paste") (roundrect_rratio 0.05494505495)
       (net 4 "Net-(J4-Pin_1)") (pinfunction "Pin_4") (pintype "passive"))
     (pad "5" smd roundrect (at -7.65 1.27 90) (size 4.6 0.8) (layers "F.Cu" "F.Paste" "F.Mask") (roundrect_rratio 0.25)
@@
   (gr_arc (start 43.18 50.8) (mid 45.411846 45.411846) (end 50.8 43.18)
     (stroke (width 0.1) (type default)) (layer "Edge.Cuts"))
+  (gr_text "GND" (at 69.85 58.42) (layer "F.SilkS")
+    (effects (font (size 1.5 1.5) (thickness 0.3) bold))
+  )
+  (gr_text "https://github.com/\nuw-madison-chem-shops/\nto263-prototype" (at 101.6 50.8) (layer "F.SilkS")
+    (effects (font (size 1.5 1.5) (thickness 0.3) bold))
+  )
   (segment (start 85.09 87.65) (end 83.84 88.9) (width 0.889) (layer "F.Cu") (net 1))
   (segment (start 73.025 88.9) (end 50.8 66.675) (width 0.889) (layer "F.Cu") (net 1))
